Commit message: update controller

File: install/bumperbot_description/share/bumperbot_description/urdf/bumperbot.urdf.xacro (robot description, xacro)
@@ -1,142 +1 @@
-<?xml version='1.0'?>
-<robot xmlns:xacro='http://www.ros.org/wiki/xacro' name='bumperbot'>
-    <xacro:arg name="is_ignition" default="true" />
-    <xacro:include filename="$(find bumperbot_description)/urdf/bumperbot_gazebo.xacro" />
-    <xacro:include filename="$(find bumperbot_description)/urdf/bumperbot_ros2_control.xacro" />
-    <link name = 'base_footprint'/>
-    <link name="base_link">
-        <inertial>
-          <origin xyz="0 0 0.04" rpy="0.0 0.25 0.3" />
-          <mass value="8.2573504e-01"/>
-          <inertia ixx="2.2124416e-02" ixy="-1.2294101e-04" ixz="3.4938785e-04"
-                   iyy="2.1193702e-02" iyz="-5.0120904e-05"
-                   izz="2.0064271e-02" />
-        </inertial>
-        <visual>
-          <origin xyz="0 0 0" rpy="0 0 0" />
-          <geometry>
-            <mesh filename="package://bumperbot_description/meshes/base_link.STL" />
-          </geometry>
-        </visual>
-        <collision>
-          <origin xyz="0 0 0" rpy="0 0 0" />
-          <geometry>
-            <mesh filename="package://bumperbot_description/meshes/base_link.STL" />
-          </geometry>
-        </collision>
-      </link>
-      <joint name="base_joint" type="fixed">
-        <parent link="base_footprint"/>
-        <child link="base_link" />
-        <origin xyz="0 0 0.033" rpy="0 0 0"/>
-      </joint>
-      <link name="wheel_right_link">
-        <inertial>
-          <origin xyz="0 -0.014 0" rpy="0 0 0" />
-          <mass value="0.0530086090966721" />
-          <inertia ixx="1.88176298336665E-05" ixy="-4.8444933029987E-10" ixz="1.88163708851143E-08"
-                   iyy="3.11510738647764E-05" iyz="-6.93560663069607E-11"
-                   izz="1.8801969558182E-05" />
-        </inertial>
-        <visual>
-          <origin xyz="0 0 0" rpy="1.57 0 0" />
-          <geometry>
-            <mesh filename="package://bumperbot_description/meshes/wheel_right_link.STL" />
-          </geometry>
-        </visual>
-        <collision>
-          <origin xyz="0 -0.015 0" rpy="1.57 0 0" />
-          <geometry>
-            <sphere radius="0.033"/>
-          </geometry>
-        </collision>
-      </link>
-      <joint name="wheel_right_joint" type="continuous">
-        <origin xyz="0 -0.0701101849418637 0" rpy="0 0 0" />
-        <parent link="base_link" />
-        <child link="wheel_right_link" />
-        <axis xyz="0 1 0" />
-      </joint>
-      <link
-        name="wheel_left_link">
-        <inertial>
-          <origin xyz="0 0.014 0" rpy="0 0 0" />
-          <mass value="0.0530086043217644" />
-          <inertia ixx="1.8792911368909E-05"  ixy="3.31256392204584E-10" ixz="-1.14082001662767E-08"
-                   iyy="3.11510738759073E-05" iyz="-3.60499245082192E-10"
-                   izz="1.88266886146847E-05" />
-        </inertial>
-        <visual>
-          <origin xyz="0 0 0" rpy="-1.57 0 0" />
-          <geometry>
-            <mesh filename="package://bumperbot_description/meshes/wheel_left_link.STL" />
-          </geometry>
-        </visual>
-        <collision>
-          <origin xyz="0 0.015 0" rpy="-1.57 0 0" />
-          <geometry>
-            <sphere radius="0.033"/>
-          </geometry>
-        </collision>
-      </link>
-      <joint name="wheel_left_joint" type="continuous">
-        <origin xyz="0 0.0701101849418642 0" rpy="0 0 0" />
-        <parent link="base_link" />
-        <child link="wheel_left_link" />
-        <axis xyz="0 1 0" />
-      </joint>
-      <link name="caster_front_link">
-        <inertial>
-          <origin xyz="3.89968128948481E-07 2.40073004698083E-07 0.00219173397061506" rpy="0 0 0" />
-          <mass value="1.44379265037903E-06" />
-          <inertia ixx="7.23075276010246E-11" ixy="-6.10956883467859E-16" ixz="2.22849693525031E-15"
-                   iyy="3.8713793085917E-11"  iyz="2.93909858781952E-15"
-                   izz="1.00967486676306E-10" />
-        </inertial>
-        <visual>
-          <origin xyz="0 0 0" rpy="0 0 0" />
-          <geometry>
-            <mesh filename="package://bumperbot_description/meshes/caster_front_link.STL" />
-          </geometry>
-        </visual>
-        <collision>
-          <origin xyz="0 0 0" rpy="0 0 0" />
-          <geometry>
-            <sphere radius="0.005"/>
-          </geometry>
-        </collision>
-      </link>
-      <joint name="caster_front_joint" type="fixed">
-        <origin xyz="0.04755 0 -0.0275" rpy="0 0 0" />
-        <parent link="base_link" />
-        <child link="caster_front_link" />
-        <axis xyz="0 0 0" />
-      </joint>
-      <link name="caster_rear_link">
-        <inertial>
-          <origin xyz="3.8996812895542E-07 2.40073004698083E-07 0.00219173397061509" rpy="0 0 0" />
-          <mass value="1.44379265037902E-06" />
-          <inertia ixx="7.23075276010246E-11" ixy="-6.10956872363424E-16" ixz="2.22849693527207E-15"
-                   iyy="3.87137930859167E-11" iyz="2.939098587861E-15"
-                   izz="1.00967486676306E-10" />
-        </inertial>
-        <visual>
-          <origin xyz="0 0 0" rpy="0 0 0" />
-          <geometry>
-            <mesh filename="package://bumperbot_description/meshes/caster_rear_link.STL" />
-          </geometry>
-        </visual>
-        <collision>
-          <origin xyz="0 0 0" rpy="0 0 0" />
-          <geometry>
-            <sphere radius="0.005"/>
-          </geometry>
-        </collision>
-      </link>
-      <joint name="caster_rear_joint" type="fixed">
-        <origin xyz="-0.04755 0 -0.0275" rpy="0 0 0" />
-        <parent link="base_link" />
-        <child link="caster_rear_link" />
-        <axis xyz="0 0 0" />
-      </joint>
-    </robot>
+/root/ros2_ws/src/bumperbot_description/urdf/bumperbot.urdf.xacro

File: install/bumperbot_description/share/bumperbot_description/urdf/bumperbot_gazebo.xacro (robot description, xacro)
@@ -1,51 +1 @@
-<?xml version="1.0"?>
-<robot name = "bumperbot" xmlns:xacro="http://www.ros.org/wiki/xacro">
-    <gazebo reference="wheel_right_link">
-        <mu1>100000000000000.0</mu1>
-        <mu2>100000000000000.0</mu2>
-        <kp>1000000000000.0</kp>
-        <kd>10.0</kd>
-        <minDepth>0.001</minDepth>
-        <maxVel>0.1</maxVel>
-        <fdir1>1 0 0</fdir1>
-    </gazebo>
-    <gazebo reference="wheel_left_link">
-        <mu1>100000000000000.0</mu1>
-        <mu2>100000000000000.0</mu2>
-        <kp>1000000000000.0</kp>
-        <kd>10.0</kd>
-        <minDepth>0.001</minDepth>
-        <maxVel>0.1</maxVel>
-        <fdir1>1 0 0</fdir1>
-    </gazebo>
-    <gazebo reference="caster_front_link">
-        <mu1>0.1</mu1>
-        <mu2>0.1</mu2>
-        <kp>1000000.0</kp>
-        <kd>100.0</kd>
-        <minDepth>0.001</minDepth>
-        <maxVel>0.1</maxVel>
-    </gazebo>
-    <gazebo reference="caster_rear_link">
-        <mu1>0.1</mu1>
-        <mu2>0.1</mu2>
-        <kp>1000000.0</kp>
-        <kd>100.0</kd>
-        <minDepth>0.001</minDepth>
-        <maxVel>0.1</maxVel>
-    </gazebo>
-    <gazebo>
-        <xacro:if value="$(arg is_ignition)">
-            <plugin filename="ign_ros2_control_system" name="ign_ros2_control::IgniteROS2ControlSystem">
-                <parameters>
-                </parameters>
-            </plugin>
-        </xacro:if>
-        <xacro:unless value="$(arg is_ignition)">
-            <plugin filename="gz_ros2_control_system" name="gz_ros2_control::GazeboSimROS2ControlSystem">
-                <parameters>
-                </parameters>
-            </plugin>
-        </xacro:unless>
-    </gazebo>
-</robot>
+/root/ros2_ws/src/bumperbot_description/urdf/bumperbot_gazebo.xacro

File: install/bumperbot_description/share/bumperbot_description/urdf/bumperbot_ros2_control.xacro (robot description, xacro)
@@ -1,31 +1 @@
-<?xml version='1.0'?>
-<robot xmlns:xacro="http://www.ros.org/wiki/xacro" name="bumperbot">
-    <ros2control name="RobotSystem" type="system">
-        <xacro:if value="$(arg is_ignition)">
-            <hardware>
-                <plugin>ign_ros2_control/IgnitionSystem</plugin>
-            </hardware>
-        </xacro:if>
-        <xacro:unless value="$(arg is_ignition)">
-            <hardware>
-                <plugin>gz_ros2_control/GazeboSimSystem</plugin>
-            </hardware>
-        </xacro:unless>
-        <joint name="wheel_right_joint">
-            <command_interface name="velocity">
-                <param name="min">-1.0</param>
-                <param name="max">1.0</param>
-            </command_interface>
-            <state_interface name="position"/>
-            <state_interface name="velocity"/>
-        </joint>
-        <joint name="wheel_left_joint">
-            <command_interface name="velocity">
-                <param name="min">-1.0</param>
-                <param name="max">1.0</param>
-            </command_interface>
-            <state_interface name="position"/>
-            <state_interface name="velocity"/>
-        </joint>
-    </ros2control>
-</robot>
+/root/ros2_ws/src/bumperbot_description/urdf/bumperbot_ros2_control.xacro

File: src/bumperbot_description/urdf/bumperbot_gazebo.xacro (robot description, xacro)
@@ -37,13 +37,11 @@
     <gazebo>
         <xacro:if value="$(arg is_ignition)">
-            <plugin filename="ign_ros2_control_system" name="ign_ros2_control::IgniteROS2ControlSystem">
-                <parameters>
-                </parameters>
+            <plugin filename="ign_ros2_control-system" name="ign_ros2_control::IgnitionROS2ControlPlugin">
+                <parameters> $(find bumperbot_controller)/config/bumperbot_controller.yaml</parameters>
             </plugin>
         </xacro:if>
         <xacro:unless value="$(arg is_ignition)">
-            <plugin filename="gz_ros2_control_system" name="gz_ros2_control::GazeboSimROS2ControlSystem">
-                <parameters>
-                </parameters>
+            <plugin filename="gz_ros2_control-system" name="gz_ros2_control::GazeboSimROS2ControlPlugin">
+                <parameters> $(find bumperbot_controller)/config/bumperbot_controller.yaml</parameters>
             </plugin>
         </xacro:unless>

File: src/bumperbot_description/urdf/bumperbot_ros2_control.xacro (robot description, xacro)
@@ -1,5 +1,5 @@
 <?xml version='1.0'?>
 <robot xmlns:xacro="http://www.ros.org/wiki/xacro" name="bumperbot">
-    <ros2control name="RobotSystem" type="system">
+    <ros2_control name="RobotSystem" type="system">
         <xacro:if value="$(arg is_ignition)">
             <hardware>
@@ -28,4 +28,4 @@
             <state_interface name="velocity"/>
         </joint>
-    </ros2control>
+    </ros2_control>
 </robot>
